Commit message: quadruped model is working in rviz

File: src/quadruped/quadruped_description/urdf/mech/leg.urdf.xacro (robot description, xacro)
@@ -1,3 +1,93 @@
 <?xml version="1.0"?>
 <robot xmlns:xacro="http://www.ros.org/wiki/xacro">
+  <xacro:macro name="leg" params="parent uid *origin">
+    <joint name="body_link1_joint_${uid}" type="revolute">
+      <parent link="${parent}"/>
+      <child link="leg_${uid}_link_1" />
+      <xacro:insert_block name="origin"/>
+      <axis xyz="0 0 1" />
+      <limit lower="${-pi/4}" upper="${pi/4}" effort="10000" velocity="10000" />
+    </joint>
+    <link name="leg_${uid}_link_1" type="revolute">
+      <visual>
+        <origin xyz="0.0 0.0 0.0"/>
+        <geometry>
+        <mesh filename="file://$(find quadruped_description)/meshes/link1.stl" />
+      </geometry>
+      <material name="cyan">
+        <color rgba="0 0.8 0.8 1" />
+      </material>
+      </visual>
+      <collision>
+      <origin xyz="-30 0 0" rpy="0 0 0" />
+      <geometry>
+        <box size="60 12 24" />
+      </geometry>
+    </collision>
+    <inertial>
+      <mass value="4" />
+      <origin xyz="0 0 0" />
+      <inertia ixx="1.0" ixy="0.0" ixz="0.0" iyy="1.0" iyz="0.0" izz="1.0" />
+    </inertial>
+    </link>
+    <joint name="leg_${uid}_joint_1" type="revolute">
+      <origin xyz="-45.955 7.75 0.045" rpy="0.0 0.0 0.0"/>
+      <parent link="leg_${uid}_link_1"/>
+      <child link="leg_${uid}_link_2"/>
+      <axis xyz="0.0 1.0 0.0"/>
+      <limit lower="${-pi/4}" upper="${pi/4}" effort="0.0" velocity="0.0"/>
+    </joint>
+    <link name="leg_${uid}_link_2">
+      <inertial>
+        <origin xyz="0.0 0.0 0.0" rpy="0.0 0.0 0.0"/>
+        <mass value="0.0"/>
+        <inertia ixx="0.0" ixy="0.0" ixz="0.0" iyy="0.0" iyz="0.0" izz="0.0"/>
+      </inertial>
+      <visual name="">
+        <origin xyz="0.0 0.0 0.0" rpy="0.0 0.0 0.0"/>
+        <geometry>
+          <mesh filename="file://$(find quadruped_description)/meshes/link2.stl" />
+        </geometry>
+        <material name="blue">
+          <color rgba="0.2 0.2 1.0 1.0"/>
+          <texture filename=""/>
+        </material>
+      </visual>
+      <collision>
+        <origin xyz="-40 0.0 0.0" rpy="0.0 0.0 0.0"/>
+        <geometry>
+          <box size="42 12 24" />
+        </geometry>
+      </collision>
+    </link>
+    <joint name="leg_${uid}_joint_2" type="revolute">
+      <parent link="leg_${uid}_link_2" />
+      <child link="leg_${uid}_feet" />
+      <origin xyz="-46.905 0 0.045" rpy="0 0 0" />
+      <axis xyz="0 1 0" />
+      <limit lower="${-2*pi/3}" upper="${pi/4}" effort="100" velocity="100" />
+    </joint>
+    <link name="leg_${uid}_feet">
+      <visual>
+        <origin xyz="0 0 0" rpy="0 0 0" />
+        <geometry>
+          <mesh filename="file://$(find quadruped_description)/meshes/link3.stl" />
+        </geometry>
+        <material name="red">
+          <color rgba="1 0.2 0.2 1" />
+        </material>
+      </visual>
+      <collision>
+        <origin xyz="-56 0 -5" rpy="0 0 0" />
+        <geometry>
+          <box size="67 12 12" />
+        </geometry>
+      </collision>
+      <inertial>
+        <mass value="1.0" />
+        <origin xyz="0 0 0" />
+        <inertia ixx="1.0" ixy="0.0" ixz="0.0" iyy="1.0" iyz="0.0" izz="1.0" />
+      </inertial>
+    </link>
+  </xacro:macro>
 </robot>

File: src/quadruped/quadruped_description/urdf/robots/quadruped.urdf.xacro (robot description, xacro)
@@ -1,5 +1,4 @@
 <?xml version="1.0"?>
 <robot xmlns:xacro="http://www.ros.org/wiki/xacro" name="quadruped">
-  <xacro:include filename="xacro_macros.urdf.xacro" />
   <link name="world"></link>
   <joint name="base_joint" type="fixed">
@@ -16,5 +15,5 @@
       </geometry>
       <material name="green">
-        <color rgba="0.2 1 0.2 1" />
+        <color rgba="0.8 0.25 0.2 1" />
       </material>
     </visual>
@@ -22,7 +21,6 @@
       <origin xyz="0 0 0" rpy="0 0 0" />
       <geometry>
-        <box size="2.5 1.5 0.1" />
-      </geometry>
-    </collision>
+        <box size="120 120 24" />
+      </geometry>q </collision>
     <inertial>
       <mass value="12" />
@@ -31,32 +29,19 @@
     </inertial>
   </link>
-  <joint name="body_link1_joint" type="revolute">
-    <parent link="robot_base_link" />
-    <child link="leg_link_1" />
-    <origin xyz="-58.77 58.981 12.432" rpy="0 0 0" />
-    <axis xyz="0 0 1" />
-    <limit lower="${-pi/4}" upper="${pi/4}" effort="10000" velocity="10000" />
-  </joint>
-  <link name="leg_link_1">
-    <visual>
-      <origin xyz="0 0 0" rpy="0 0 0" />
-      <geometry>
-        <mesh filename="file://$(find quadruped_description)/meshes/link1.stl" />
-      </geometry>
-      <material name="cyan">
-        <color rgba="0 1 1 1" />
-      </material>
-    </visual>
-    <collision>
-      <origin xyz="0 0 0" rpy="0 0 0" />
-      <geometry>
-        <box size="1 2 1" />
-      </geometry>
-    </collision>qq
-    <inertial>
-      <mass value="4" />
-      <origin xyz="0 0 0" />
-      <inertia ixx="1.0" ixy="0.0" ixz="0.0" iyy="1.0" iyz="0.0" izz="1.0" />
-    </inertial>
-  </link>
+  <xacro:include filename="$(find quadruped_description)/urdf/mech/leg.urdf.xacro" />
+  <xacro:leg parent="robot_base_link" uid="fr">
+    <origin xyz="-58.77 58.981 12.432" rpy="0 0 ${-pi/4}"/>
+  </xacro:leg>
+  <xacro:include filename="$(find quadruped_description)/urdf/mech/leg.urdf.xacro" />
+  <xacro:leg parent="robot_base_link" uid="fl">
+    <origin xyz="58.77 58.981 12.432" rpy="0 0 ${-3*pi/4}"/>
+  </xacro:leg>
+  <xacro:include filename="$(find quadruped_description)/urdf/mech/leg.urdf.xacro" />
+  <xacro:leg parent="robot_base_link" uid="br">
+    <origin xyz="-58.77 -58.981 12.432" rpy="0 0 ${pi/4}"/>
+  </xacro:leg>
+  <xacro:include filename="$(find quadruped_description)/urdf/mech/leg.urdf.xacro" />
+  <xacro:leg parent="robot_base_link" uid="bl">
+    <origin xyz="58.77 -58.981 12.432" rpy="0 0 ${3*pi/4}"/>
+  </xacro:leg>
 </robot>
